Commit message: Remove trailing slash from mesh URI paths
The meshes_file_direction xacro property ended with a slash while
every <mesh filename> reference adds its own, producing URIs like
package://open_manipulator_description/meshes/omy_f3m//base_unit.stl.

The double slash fails foxglove_bridge's default asset_uri_allowlist
regex (empty path segments do not match), so Foxglove cannot fetch
the meshes and the robot model renders without geometry. RViz
tolerates the double slash, which is why this went unnoticed.

Backport of upstream ROBOTIS-GIT/open_manipulator commit 29b52de1,
which applies the identical fix to omx_f, omx_l, omy_3m, omy_f3m,
and omy_l100.

Co-Authored-By: Claude Fable 5 <noreply@anthropic.com>

File: open_manipulator_description/urdf/omy_f3m/omy_f3m_arm.urdf.xacro (robot description, xacro)
@@ -2,5 +2,5 @@
 <robot xmlns:xacro="http://www.ros.org/wiki/xacro">
    <xacro:macro name="omy_f3m" params="prefix">
-      <xacro:property name="meshes_file_direction" value="package://open_manipulator_description/meshes/omy_f3m/" />
+      <xacro:property name="meshes_file_direction" value="package://open_manipulator_description/meshes/omy_f3m" />
       <link name="${prefix}link0">
          <visual>
